File: digirig_icom.kicad_pcb (KiCad board)
At the start: 4 copper layers, 48.5 x 56 mm, 64 parts, among them CON2 SJ-3523-SMT-TR, IC1 RP2354, J1 RJ45, J2 RJ45, J3 USB_B, Q1 AO3401A, Q2 2N7002, Q3 MMBT3904, Q4 MMBT3904, SW1 SW_SPST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

Commit message: Weird level shifting stuff I think
Parts:
- added R16: 47k, Resistor_SMD:R_0402_1005Metric, B.Cu at (13.8, 57.1)
- added R17: 12k, Resistor_SMD:R_0402_1005Metric, B.Cu at (15.3, 59.5)
- added R18: 1k, Resistor_SMD:R_0402_1005Metric, B.Cu at (27.5, 53.6)
- added R19: 100k, Resistor_SMD:R_0402_1005Metric, B.Cu at (23.1, 53.1)
- added U5: LM393DR, digikey-footprints:SOIC-8_W3.9mm, B.Cu at (17.7, 53.2)
- added U6: TXS0102DQE, Package_SON:X2SON-8_1.4x1mm_P0.35mm, B.Cu at (32.1, 56.9)
- moved C21 2.01 mm to (29.4, 46.8), turned to 180 degrees
Connections:
- IC1 pad 15: /DATA_MCU -> unconnected-(IC1-GPIO11-Pad15)
- IC1 pad 40: unconnected-(IC1-GPIO26_ADC0-Pad40) -> /DATA_MCU_IN
- IC1 pad 41: unconnected-(IC1-GPIO27_ADC1-Pad41) -> /DATA_MCU_OUT
Routing:
- net /DATA_H: track 26.2 -> 55.2 mm, vias 2 -> 3
- net +5V: track 24.1 -> 50.1 mm
- net /DATA_MCU: track 16.0 -> 34.5 mm, vias 0 -> 4
- net Net-(R18-Pad2): track 0.00 -> 18.3 mm
- net /DATA_MCU_OUT: track 0.00 -> 17.9 mm, vias 0 -> 2
- net /DATA_MCU_IN: track 0.00 -> 17.8 mm, vias 0 -> 2
- net Net-(R16-Pad1): track 0.00 -> 8.69 mm
- net +3V3: track 44.0 -> 51.1 mm, vias 13 -> 16
- net GND: track 44.5 -> 44.9 mm, vias 39 -> 40

Commit message: Fix some stuff
Parts:
- C1, C12, C13, C14, C15, C16, C17, C18, C19, C2, C3: footprint Capacitor_SMD:C_0201_0603Metric -> Capacitor_SMD:C_0402_1005Metric
