File: digirig_icom.kicad_sch (KiCad schematic)
At the start: 60 parts, among them CON2 SJ-3523-SMT-TR, IC1 RP2354, J1 RJ45, J2 RJ45, J3 USB_B, Q1 AO3401A, Q2 2N7002, Q3 MMBT3904, Q4 MMBT3904, SW1 SW_SPST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

Commit message: Weird level shifting stuff I think
Parts:
- added R16: 47k, Resistor_SMD:R_0402_1005Metric, symbol Device:R
- added R17: 12k, Resistor_SMD:R_0402_1005Metric, symbol Device:R
- added R18: 1k, Resistor_SMD:R_0402_1005Metric, symbol Device:R
- added R19: 100k, Resistor_SMD:R_0402_1005Metric, symbol Device:R
- added U5: LM393DR, digikey-footprints:SOIC-8_W3.9mm, symbol dk_Linear-Comparators:LM393DR
- added U6: TXS0102DQE, Package_SON:X2SON-8_1.4x1mm_P0.35mm, symbol Logic_LevelTranslator:TXS0102DQE
Connections:
- net +3V3: now also U5.8 (VCC), U6.1 (VCCA), U6.5 (OE)
- net +5V: now also R17.1, U6.8 (VCCB)
- net DATA_H: now also R18.1
- net DATA_MCU: now also U6.7 (B1); no longer IC1.15 (GPIO11)
- net GND: now also R16.2, U5.4 (GND), U6.4 (GND)
- net DATA_MCU_IN: now reaches IC1.40 (GPIO26_ADC0)
- net DATA_MCU_IN: now also R19.2, U5.1 (1OUT)
- net DATA_MCU_OUT: now reaches IC1.41 (GPIO27_ADC1)
- net DATA_MCU_OUT: now also U6.2 (A1)
- new net: R16.1, R17.2, U5.2
- new net: R18.2, R19.1, U5.3
- no-connect marks 36 -> 37
Other:
- note added: "Level shifting tx"
- note added: "Weird rx level shifting"
- moved on the sheet: C16, R7, R8

Commit message: Fix some stuff
Parts:
- C1, C12, C13, C14, C15, C16, C17, C2, C3: footprint Capacitor_SMD:C_0201_0603Metric -> Capacitor_SMD:C_0402_1005Metric; Digi-Key_PN (none) -> 1276-1482-2-ND
- C10, C8: Digi-Key_PN (none) -> 490-6186-2-ND
- C11, C20, C21, C4, C5, C6, C9: Digi-Key_PN (none) -> 1276-1043-2-ND
- C18, C19: footprint Capacitor_SMD:C_0201_0603Metric -> Capacitor_SMD:C_0402_1005Metric; Digi-Key_PN (none) -> 1276-1010-2-ND
- D1, D2: Digi-Key_PN (none) -> SS14TR-ND
- D3: Digi-Key_PN (none) -> 475-LSQ976-NR-1TR-ND
- IC1: Digi-Key_PN (none) -> 2648-SC1511(13)-A4TR-ND
- J1, J2: Digi-Key_PN (none) -> 609-1046-ND
- J3: Digi-Key_PN (none) -> 5405-241106-ND
- L1: Digi-Key_PN (none) -> 535-AOTA-B201610S3R3-101-TTR-ND
- Q3, Q4: Digi-Key_PN (none) -> 4878-MMBT3904TR-ND
- R1: Digi-Key_PN (none) -> 311-33JRTR-ND
- R10, R18, R3, R4, R8: Digi-Key_PN (none) -> 311-1.0KJRTR-ND
- R11, R12: Digi-Key_PN (none) -> 311-22.0LRTR-ND
- R13, R14, R2, R5, R7, R9: Digi-Key_PN (none) -> 311-10.0KLRTR-ND
- R15: Digi-Key_PN (none) -> 311-220HRTR-ND
- R16: Digi-Key_PN (none) -> 311-47.0KLRTR-ND
- R17: Digi-Key_PN (none) -> P12KDCTR-ND
- R19: Digi-Key_PN (none) -> 311-100KJRTR-ND
- R6: Digi-Key_PN (none) -> 311-470LRTR-ND
- SW1: Digi-Key_PN (none) -> CKN10384TR-ND
- U1: Digi-Key_PN (none) -> 296-23775-2-ND
- U2, U3: Digi-Key_PN (none) -> 296-14117-2-ND
- U4: Digi-Key_PN (none) -> MCP1703A-3302E/DB-ND
- U6: Digi-Key_PN (none) -> 296-28368-2-ND
- Y1: Digi-Key_PN (none) -> 535-ABM8-272-T3TR-ND
